Commit message: zed: add base tutorial zed launcher with scoutM bot scout: - Added some todos to check up on before actual launch (PCL node should be moved) FRANCIS: - up a bunch of launcher files

File: zed_robot_integration/urdf/zed_robot_mono.urdf.xacro (robot description, xacro)
@@ -1,50 +1,37 @@
 <?xml version="1.0"?>
-<!--
-// Copyright 2024 Stereolabs
-//
-// Licensed under the Apache License, Version 2.0 (the "License");
-// you may not use this file except in compliance with the License.
-// You may obtain a copy of the License at
-//
-//      http://www.apache.org/licenses/LICENSE-2.0
-//
-// Unless required by applicable law or agreed to in writing, software
-// distributed under the License is distributed on an "AS IS" BASIS,
-// WITHOUT WARRANTIES OR CONDITIONS OF ANY KIND, either express or implied.
-// See the License for the specific language governing permissions and
-// limitations under the License.
--->
-<robot name="zedbot_scoutm" xmlns:xacro="http://ros.org/wiki/xacro">
-  <xacro:arg name="camera_name"   default="zed" />
-  <xacro:arg name="camera_model"  default="zedx" />
-  <xacro:arg name="use_zed_localization" default="true" />
-  <xacro:arg name="baseline" default="0.0" />
-  <!-- Include the robot (e.g. AgileX Scout mini) -->
-  <xacro:include filename="$(find scout_description)/urdf/scout_mini.xacro" />
-  <!-- Add one ZED Camera -->
-  <xacro:include filename="$(find zed_wrapper)/urdf/zed_macro.urdf.xacro" />
-  <xacro:zed_camera name="$(arg camera_name)" model="$(arg camera_model)" baseline="$(arg baseline)"/>
-  <!-- Add a joint to connect the ZED Camera to the robot -->
-  <xacro:if value="$(arg use_zed_localization)">
-    <!-- ZED Localization -> The reference link is '$(arg camera_name)_camera_link' and 'base_link' is a child -->
-    <joint name="$(arg camera_name)_joint" type="fixed">
-      <parent link="$(arg camera_name)_camera_link"/>
-      <child link="base_link"/>
-      <origin
-        xyz="-0.12 0.0 -0.25"
-        rpy="0 0 0"
-      />
-    </joint>
-  </xacro:if>
-  <xacro:unless value="$(arg use_zed_localization)">
-    <!-- NO ZED Localization -> '$(arg camera_name)_camera_link' is a child of 'base_link' -->
-    <joint name="$(arg camera_name)_joint" type="fixed">
-      <parent link="base_link"/>
-      <child link="$(arg camera_name)_camera_link"/>
-      <origin
-        xyz="0.12 0.0 0.25"
-        rpy="0 0 0"
-      />
-    </joint>
-  </xacro:unless>
+<robot name="scoutm" xmlns:xacro="http://ros.org/wiki/xacro">
+    <xacro:arg name="camera_name" default="zed"/>
+    <xacro:arg name="camera_model" default="zed2i"/>
+    <xacro:arg name="use_zed_localization" default="true"/>
+    <xacro:arg name="baseline" default="0.0"/>
+    <!-- Include the robot (e.g. AgileX Scout mini) -->
+    <xacro:include filename="$(find scout_description)/urdf/scout2.urdf.xacro"/>
+    <!-- Add one ZED Camera -->
+    <xacro:include filename="$(find zed_wrapper)/urdf/zed_macro.urdf.xacro"/>
+    <xacro:zed_camera name="$(arg camera_name)" model="$(arg camera_model)" custom_baseline="$(arg baseline)">
+        <gnss_origin/>
+    </xacro:zed_camera>
+    <!-- Add a joint to connect the ZED Camera to the robot -->
+    <xacro:if value="$(arg use_zed_localization)">
+        <!-- ZED Localization -> The reference link is '$(arg camera_name)_camera_link' and 'base_link' is a child -->
+        <joint name="$(arg camera_name)_joint" type="fixed">
+            <parent link="$(arg camera_name)_camera_link"/>
+            <child link="base_link"/>
+            <origin
+                    xyz="-0.12 0.0 -0.25"
+                    rpy="0 0 0"
+            /><!--todo update with new pos-->
+        </joint>
+    </xacro:if>
+    <xacro:unless value="$(arg use_zed_localization)"><!--we arent using this so don't rly need to worry about it-->
+        <!-- NO ZED Localization -> '$(arg camera_name)_camera_link' is a child of 'base_link' -->
+        <joint name="$(arg camera_name)_joint" type="fixed">
+            <parent link="base_link"/>
+            <child link="$(arg camera_name)_camera_link"/>
+            <origin
+                    xyz="0.12 0.0 0.25"
+                    rpy="0 0 0"
+            />
+        </joint>
+    </xacro:unless>
 </robot>

Commit message: zed: - take out PCL node since we want 3d scans - simplify urdf file
scout:
- take out laser frame gazebo ref in ouster
- scout_mini_base.launch.py clean imports
- add uT lidar stl but its too big lol

File: zed_robot_integration/urdf/zed_robot_mono.urdf.xacro (robot description, xacro)
@@ -2,8 +2,8 @@
 <robot name="scoutm" xmlns:xacro="http://ros.org/wiki/xacro">
     <xacro:arg name="camera_name" default="zed"/>
-    <xacro:arg name="camera_model" default="zed2i"/>
-    <xacro:arg name="use_zed_localization" default="true"/>
+    <xacro:arg name="camera_model" default="zed"/>
+    <xacro:arg name="use_zed_localization" default="false"/>
     <xacro:arg name="baseline" default="0.0"/>
-    <!-- Include the robot (e.g. AgileX Scout mini) -->
+    <!-- AgileX Scout mini + Lidar_base -->
     <xacro:include filename="$(find scout_description)/urdf/scout2.urdf.xacro"/>
     <!-- Add one ZED Camera -->
@@ -12,26 +12,28 @@
         <gnss_origin/>
     </xacro:zed_camera>
-    <!-- Add a joint to connect the ZED Camera to the robot -->
+    <joint name="$(arg camera_name)_joint" type="fixed">
+        <parent link="base_link"/>
+        <child link="$(arg camera_name)_camera_link"/>
+        <origin
+                xyz="0.3 0.0 0"
+                rpy="0 0 0"
+        />
+    </joint>
+<!--    &lt;!&ndash; Add a joint to connect the ZED Camera to the robot  &ndash;&gt;
     <xacro:if value="$(arg use_zed_localization)">
-        <!-- ZED Localization -> The reference link is '$(arg camera_name)_camera_link' and 'base_link' is a child -->
+        &lt;!&ndash; We really don't care about this part since we never use zed's localizer since we're using robot_localization instead
+        ZED Localization -> The reference link is '$(arg camera_name)_camera_link' and 'base_link' is a child &ndash;&gt;
         <joint name="$(arg camera_name)_joint" type="fixed">
             <parent link="$(arg camera_name)_camera_link"/>
             <child link="base_link"/>
             <origin
-                    xyz="-0.12 0.0 -0.25"
+                    xyz="1 0.0 -.5"
                     rpy="0 0 0"
-            /><!--todo update with new pos-->
+            />&lt;!&ndash;todo update with new pos&ndash;&gt;
         </joint>
     </xacro:if>
-    <xacro:unless value="$(arg use_zed_localization)"><!--we arent using this so don't rly need to worry about it-->
-        <!-- NO ZED Localization -> '$(arg camera_name)_camera_link' is a child of 'base_link' -->
-        <joint name="$(arg camera_name)_joint" type="fixed">
-            <parent link="base_link"/>
-            <child link="$(arg camera_name)_camera_link"/>
-            <origin
-                    xyz="0.12 0.0 0.25"
-                    rpy="0 0 0"
-            />
-        </joint>
-    </xacro:unless>
+    <xacro:unless value="$(arg use_zed_localization)">
+        &lt;!&ndash; NO ZED Localization -> '$(arg camera_name)_camera_link' is a child of 'base_link' &ndash;&gt;
+        &lt;!&ndash;original joint code goes here&ndash;&gt;
+    </xacro:unless>-->
 </robot>
